Commit message: Fixes: - completed removal of sensor frame inversion - Ethernet / CAN parsing of sensor data - improved sample buckets splitting first shuffle then split uniformly) - added last 'averageOptimalDq' just for evaluating the improvement due   to the joints offsets - cost computation after optimisation: removed rad/degrees conversion - plotting auto-scale - fixed left, right legs sensor frames in URDF model

File: src/models/iCubGenova02/iCubFull.urdf (robot description, URDF)
Before this commit: robot iCubGenova02, 105 links, 104 joints
Joints:
- joint l_lower_leg_mtb_acc_10b10_fixed_joint: origin xyz=0.030989 -0.011037 0.05238133 rpy=-1.32645042367 0 1.57079632679 -> xyz=0.0665272 -0.043468 0.0259151 rpy=1.30899714594 -0.000112159802878 1.57082638021
- joint l_lower_leg_mtb_acc_10b8_fixed_joint: origin xyz=0.0099841 -0.004318 0.0544518 rpy=-0.349065638045 3.97141037841e-05 1.57090544048 -> xyz=0.030989 -0.011037 0.05238133 rpy=0.2426 0 1.5708
- joint l_lower_leg_mtb_acc_10b9_fixed_joint: origin xyz=0.0665272 -0.043468 0.0259151 rpy=1.30899714594 -0.000112159802878 1.57082638021 -> xyz=0.0099841 -0.004318 0.0544518 rpy=-0.349065638045 3.97141037841e-05 1.57090544048
- joint l_upper_leg_mtb_acc_10b2_fixed_joint: origin xyz=0.0083839 0.039452 0.05335544 rpy=0.837758036965 -8.62912869137e-05 1.57087402394 -> xyz=0.0083839 0.039452 0.05335544 rpy=0.2618 0 1.5709
- joint r_lower_leg_mtb_acc_11b10_fixed_joint: origin xyz=-0.0389997 -0.004318 0.05362922 rpy=-0.244346164565 2.80911040962e-05 1.57090899435 -> xyz=-0.0660179 -0.043468 0.0278945 rpy=-1.3089971473150512 0 1.5707963267948968
- joint r_lower_leg_mtb_acc_11b8_fixed_joint: origin xyz=-0.008081 -0.004318 0.0537517 rpy=0.349065638046 -3.97141043948e-05 1.57090544048 -> xyz=-0.0389997 -0.004318 0.05362922 rpy=-0.2443461645654741 2.8091104096089837e-05 1.5709089943462522
- joint r_lower_leg_mtb_acc_11b9_fixed_joint: origin xyz=-0.0660179 -0.043468 0.0278945 rpy=-1.30899714732 0 1.57079632679 -> xyz=-0.008081 -0.004318 0.0537517 rpy=0.34906563804609786 -3.971410439477034e-05 1.5709054404832665
- joint r_upper_leg_mtb_acc_11b2_fixed_joint: origin xyz=-0.0064065 0.039256 0.0539467 rpy=-0.837758053858 -0.000342790749344 1.57087401652 -> xyz=-0.0064065 0.039256 0.0539467 rpy=-0.2618 0 1.57087
